File: 10-pcb-power/pcb_power/pcb_power.kicad_pcb (KiCad board)
At the start: 2 copper layers, 8 parts, among them J1 Pwr_jmp, U1 RP402N331F

Commit message: Power Layout
Parts:
- added BT1: Battery, Battery:BatteryHolder_TruPower_BH-331P_3xAA, F.Cu at (179.1, 123.6)
- added SW1: SW_SPDT, Button_Switch_SMD:SW_SPDT_CK-JS102011SAQN, F.Cu at (170.7, 110.5)
- moved TP1 15.5 mm to (163.8, 102.9), turned to 90 degrees
- moved J1 13.9 mm to (159.3, 104.1), turned to 0 degrees
- moved JP1 13.5 mm to (156.1, 106.4), turned to 90 degrees
- moved L1 10.8 mm to (163.8, 106.4), turned to 90 degrees
- moved C1 4.44 mm to (164.6, 110.7), turned to -90 degrees
- moved U1 2.16 mm to (161.4, 111.0)
Connections:
- net Net-(L1-Pad2) renamed /vreg_lx
- U1 pad 3: power_en -> /vreg_en
Routing:
- net /vreg_en: track 0.00 -> 7.45 mm
- net /vreg_lx: track 0.00 -> 2.51 mm, vias 0 -> 8
- added copper zone on F.Cu, net +BATT
- added copper zone on B.Cu, net /vreg_lx
- added copper zone on F.Cu, net /vreg_lx
- added copper zone on F.Cu, net /vreg_out
- added copper zone on F.Cu, net GND

Commit message: More PCB Work
Parts:
- added C4: C_Small, Capacitor_SMD:C_0805_2012Metric, F.Cu at (168.9, 94.5)
- added D1: LED, LED_SMD:LED_0805_2012Metric, F.Cu at (161.5, 66.8)
- added J2: CPU_jmp, Connector_PinHeader_2.54mm:PinHeader_1x02_P2.54mm_Vertical, F.Cu at (165.0, 94.5)
- added J3: Serial Header, Connector_PinHeader_2.54mm:PinHeader_1x04_P2.54mm_Vertical, F.Cu at (155.8, 111.0)
- added J4: Programming Header, Connector_PinHeader_2.54mm:PinHeader_1x04_P2.54mm_Vertical, F.Cu at (155.8, 98.3)
- added JP2: CPU_jmp, Jumper:SolderJumper-2_P1.3mm_Open_TrianglePad1.0x1.5mm, F.Cu at (161.8, 95.6)
- added R1: R_Small_US, Resistor_SMD:R_0805_2012Metric, F.Cu at (155.4, 70.4)
- added R2: R_Small_US, Resistor_SMD:R_0805_2012Metric, F.Cu at (157.5, 70.4)
- added R3: R_Small_US, Resistor_SMD:R_0805_2012Metric, F.Cu at (159.5, 70.4)
- added R4: R_Small_US, Resistor_SMD:R_0805_2012Metric, F.Cu at (161.5, 70.4)
- added SW2: SW_SPST, Button_Switch_SMD:SW_SPST_CK_RS282G05A3, F.Cu at (174.8, 90.2)
- added SW3: SW_SPST, Button_Switch_SMD:SW_SPST_CK_RS282G05A3, F.Cu at (174.8, 69.8)
- added SW4: SW_SPST, Button_Switch_SMD:SW_SPST_CK_RS282G05A3, F.Cu at (174.8, 80.0)
- added U2: LoRa-E5, LoRa-E5:LoRa-E5, F.Cu at (164.6, 83.6)
- added U3: IN-S128TATRGB, RGB_LED:IN-S128TATRGB, F.Cu at (154.6, 65.2)
- moved BT1 9.15 mm to (188.2, 123.8)
- moved JP1 6.81 mm to (161.8, 102.7)
- moved C2 6.25 mm to (161.8, 108.2)
- moved C3 6.25 mm to (164.0, 108.2)
- moved J1 6.25 mm to (165.0, 101.6)
- moved U1 6.25 mm to (167.1, 108.5)
- moved SW1 6.25 mm to (176.4, 108.0)
- moved C1 6.25 mm to (170.3, 108.2)
- moved L1 6.25 mm to (169.5, 103.9)
- moved TP1 6.25 mm to (169.5, 100.3)
Routing:
- net TX/PB6: track 0.00 -> 40.2 mm, vias 0 -> 1
- net RX/PB7: track 0.00 -> 37.3 mm, vias 0 -> 1
- net +3V3: track 0.00 -> 34.2 mm
- net SWCLK/PA14: track 0.00 -> 18.2 mm, vias 0 -> 1
- net LED_R: track 0.00 -> 17.9 mm
- net LED_G: track 0.00 -> 17.6 mm
- net LED_B: track 0.00 -> 17.3 mm
- net SWDIO/PA13: track 0.00 -> 16.4 mm, vias 0 -> 1
- net Net-(R3-Pad2): track 0.00 -> 4.27 mm
- net Net-(R2-Pad2): track 0.00 -> 2.67 mm
- net Net-(R1-Pad2): track 0.00 -> 2.06 mm
- net Net-(D1-Pad2): track 0.00 -> 1.71 mm
- net BOOT/PB13: track 0.00 -> 0.91 mm
- net RST: track 0.00 -> 0.84 mm
- net PA0/BUTTON: track 0.00 -> 0.73 mm
- added copper zone on F.Cu, net +3V3
- added copper zone on F.Cu, net Vcc
Other:
- board outline added: 25.4 x 50.8 mm
