File: pcb_power/pcb_power.kicad_sch (KiCad schematic)
At the start: 26 parts, among them J1 Pwr_jmp, J2 CPU_jmp, J3 Serial Header, J4 Programming Header, SW1 SW_SPDT, SW2 SW_SPST, SW3 SW_SPST, SW4 SW_SPST, U1 RP402N331F, U2 LoRa-E5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

Commit message: Changes
Parts:
- added C5: 10u, Capacitor_SMD:C_0805_2012Metric, symbol Device:C_Small
- added CR1: STTS75M2F, STTS75M2F:STTS75M2F, symbol STTS75M2F:STTS75M2F
- added R5, R6, R7: 10k, Resistor_SMD:R_0805_2012Metric, symbol Device:R_Small_US
- AE1: footprint (none) -> Connector_Coaxial:U.FL_Molex_MCRF_73412-0110_Vertical
- BT1: footprint Connector_PinHeader_1.00mm:PinHeader_1x02_P1.00mm_Vertical -> Connector_PinHeader_2.54mm:PinHeader_1x02_P2.54mm_Horizontal
Connections:
- net +3V3: now also C5.1, CR1.8 (VDD), R5.1, R6.1, R7.1
- net GND: now also C5.2, CR1.4 (GND), CR1.5 (A2), CR1.6 (A1), CR1.7 (A0)
- net PA15/SDA: now also CR1.1 (SDA), R5.2
- net PB15/SCL: now also CR1.2 (SCL), R6.2
- new net: CR1.3 (*OS/INT), R7.2

Commit message: DRC Fixes, etc
Parts:
- added J5: Pins Header, Connector_PinHeader_2.54mm:PinHeader_1x04_P2.54mm_Vertical_SMD_Pin1Left, symbol Connector:Conn_01x04_Male
- added JP3: OSINT_Jmp, Jumper:SolderJumper-2_P1.3mm_Bridged2Bar_Pad1.0x1.5mm, symbol Jumper:SolderJumper_2_Open
Connections:
- net +3V3: no longer J4.2 (Pin_2)
- net RST: now also J4.2 (Pin_2)
- net PA3: now reaches U2.18 (PA3)
- net PA3: now also J5.4 (Pin_4)
- net PA2: now reaches U2.19 (PA2)
- net PA2: now also J5.2 (Pin_2)
- net PB10: now reaches U2.20 (PB10)
- net PB10: now also J5.3 (Pin_3)
- net PA9: now reaches U2.21 (PA9)
- net PA9: now also J5.1 (Pin_1), JP3.1 (A)
- net at CR1.3 (*OS/INT), R7.2: now also JP3.2 (B)
- no-connect marks 10 -> 6

Commit message: Add files via upload
Parts:
- added C6, C7: C, Capacitor_SMD:C_0603_1608Metric_Pad1.08x0.95mm_HandSolder, symbol Device:C
- added R8, R9: R, Resistor_SMD:R_0603_1608Metric_Pad0.98x0.95mm_HandSolder, symbol Device:R
Connections:
- net GND: now also C6.2, C7.2
- net RFIO: now also C6.1, R8.1; no longer AE1.1 (A)
- new net: C7.1, R8.2, R9.1
- new net: AE1.1 (A), R9.2
Other:
- moved on the sheet: AE1
Changed lines of the file:
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@@
   (junction (at 88.9 38.1) (diameter 0) (color 0 0 0 0)
   )
+  (junction (at 88.9 175.26) (diameter 0) (color 0 0 0 0)
+  )
   (junction (at 116.84 38.1) (diameter 0) (color 0 0 0 0)
+  )
+  (junction (at 97.79 175.26) (diameter 0) (color 0 0 0 0)
+  )
+  (junction (at 88.9 163.83) (diameter 0) (color 0 0 0 0)
   )
   (junction (at 53.34 35.56) (diameter 0) (color 0 0 0 0)
@@
   (no_connect (at 81.28 137.16))
   (no_connect (at 78.74 137.16))
+  (wire (pts (xy 88.9 163.83) (xy 90.17 163.83))
+    (stroke (width 0) (type default) (color 0 0 0 0))
+  )
   (wire (pts (xy 241.3 45.72) (xy 241.3 48.26))
     (stroke (width 0) (type default) (color 0 0 0 0))
@@
     (stroke (width 0) (type default) (color 0 0 0 0))
   )
-  (wire (pts (xy 91.44 163.83) (xy 92.71 163.83))
-    (stroke (width 0) (type default) (color 0 0 0 0))
-  )
   (wire (pts (xy 187.96 55.88) (xy 185.42 55.88))
     (stroke (width 0) (type default) (color 0 0 0 0))
@@
     (stroke (width 0) (type default) (color 0 0 0 0))
   )
+  (wire (pts (xy 97.79 175.26) (xy 97.79 166.37))
+    (stroke (width 0) (type default) (color 0 0 0 0))
+  )
   (wire (pts (xy 116.84 38.1) (xy 116.84 43.18))
     (stroke (width 0) (type default) (color 0 0 0 0))
@@
     (stroke (width 0) (type default) (color 0 0 0 0))
   )
+  (wire (pts (xy 88.9 175.26) (xy 97.79 175.26))
+    (stroke (width 0) (type default) (color 0 0 0 0))
+  )
   (wire (pts (xy 93.98 119.38) (xy 95.25 119.38))
     (stroke (width 0) (type default) (color 0 0 0 0))
@@
     (stroke (width 0) (type default) (color 0 0 0 0))
   )
+  (wire (pts (xy 81.28 167.64) (xy 81.28 163.83))
+    (stroke (width 0) (type default) (color 0 0 0 0))
+  )
   (wire (pts (xy 57.15 119.38) (xy 58.42 119.38))
     (stroke (width 0) (type default) (color 0 0 0 0))
@@
     (stroke (width 0) (type default) (color 0 0 0 0))
   )
+  (wire (pts (xy 88.9 163.83) (xy 88.9 167.64))
+    (stroke (width 0) (type default) (color 0 0 0 0))
+  )
   (wire (pts (xy 114.3 138.43) (xy 116.84 138.43))
     (stroke (width 0) (type default) (color 0 0 0 0))
@@
     (stroke (width 0) (type default) (color 0 0 0 0))
   )
+  (wire (pts (xy 81.28 163.83) (xy 80.01 163.83))
+    (stroke (width 0) (type default) (color 0 0 0 0))
+  )
   (wire (pts (xy 121.92 76.2) (xy 120.65 76.2))
     (stroke (width 0) (type default) (color 0 0 0 0))
@@
     (stroke (width 0) (type default) (color 0 0 0 0))
   )
-  (wire (pts (xy 92.71 167.64) (xy 92.71 166.37))
+  (wire (pts (xy 97.79 177.8) (xy 97.79 175.26))
     (stroke (width 0) (type default) (color 0 0 0 0))
   )
@@
   )
   (wire (pts (xy 58.42 95.25) (xy 48.26 95.25))
+    (stroke (width 0) (type default) (color 0 0 0 0))
+  )
+  (wire (pts (xy 81.28 175.26) (xy 88.9 175.26))
     (stroke (width 0) (type default) (color 0 0 0 0))
   )
@@
     )
   )
-  (global_label "RFIO" (shape input) (at 91.44 163.83 180) (fields_autoplaced)
-    (effects (font (size 1 1)) (justify right))
-    (property "Intersheet References" "${INTERSHEET_REFS}" (id 0) (at 86.159 163.7675 0)
+  (global_label "RFIO" (shape input) (at 80.01 163.83 180) (fields_autoplaced)
+    (effects (font (size 1 1)) (justify right))
+    (property "Intersheet References" "${INTERSHEET_REFS}" (id 0) (at 74.729 163.7675 0)
       (effects (font (size 1 1)) (justify right) hide)
     )
@@
     (pin "1")
   )
+  (symbol (lib_id "Device:R") (at 93.98 163.83 90) (unit 1)
+    (in_bom yes) (on_board yes) (fields_autoplaced)
+    (property "Reference" "R9" (id 0) (at 93.98 157.48 90))
+    (property "Value" "R" (id 1) (at 93.98 160.02 90))
+    (property "Footprint" "Resistor_SMD:R_0603_1608Metric_Pad0.98x0.95mm_HandSolder" (id 2) (at 93.98 165.608 90)
+      (effects (font (size 1.27 1.27)) hide)
+    )
+    (property "Datasheet" "~" (id 3) (at 93.98 163.83 0)
+      (effects (font (size 1.27 1.27)) hide)
+    )
+    (pin "1")
+    (pin "2")
+  )
   (symbol (lib_id "power:+3V3") (at 53.34 175.26 0) (unit 1)
     (in_bom yes) (on_board yes) (fields_autoplaced)
@@
     (pin "1")
   )
+  (symbol (lib_id "Device:C") (at 88.9 171.45 0) (unit 1)
+    (in_bom yes) (on_board yes) (fields_autoplaced)
+    (property "Reference" "C7" (id 0) (at 92.71 170.1799 0)
+      (effects (font (size 1.27 1.27)) (justify left))
+    )
+    (property "Value" "C" (id 1) (at 92.71 172.7199 0)
+      (effects (font (size 1.27 1.27)) (justify left))
+    )
+    (property "Footprint" "Capacitor_SMD:C_0603_1608Metric_Pad1.08x0.95mm_HandSolder" (id 2) (at 89.8652 175.26 0)
+      (effects (font (size 1.27 1.27)) hide)
+    )
+    (property "Datasheet" "~" (id 3) (at 88.9 171.45 0)
+      (effects (font (size 1.27 1.27)) hide)
+    )
+    (pin "1")
+    (pin "2")
+  )
   (symbol (lib_id "Device:R_Small_US") (at 35.56 154.94 90) (unit 1)
     (in_bom yes) (on_board yes) (fields_autoplaced)
@@
     (pin "2")
   )
-  (symbol (lib_id "Device:Antenna_Shield") (at 97.79 163.83 270) (unit 1)
-    (in_bom yes) (on_board yes) (fields_autoplaced)
-    (property "Reference" "AE1" (id 0) (at 104.14 163.1314 90)
-      (effects (font (size 1.27 1.27)) (justify left))
-    )
-    (property "Value" "Antenna_Shield" (id 1) (at 104.14 165.6714 90)
-      (effects (font (size 1.27 1.27)) (justify left))
-    )
-    (property "Footprint" "Connector_Coaxial:U.FL_Molex_MCRF_73412-0110_Vertical" (id 2) (at 100.33 163.83 0)
-      (effects (font (size 1.27 1.27)) hide)
-    )
-    (property "Datasheet" "~" (id 3) (at 100.33 163.83 0)
+  (symbol (lib_id "Device:Antenna_Shield") (at 102.87 163.83 270) (unit 1)
+    (in_bom yes) (on_board yes) (fields_autoplaced)
+    (property "Reference" "AE1" (id 0) (at 109.22 163.1314 90)
+      (effects (font (size 1.27 1.27)) (justify left))
+    )
+    (property "Value" "Antenna_Shield" (id 1) (at 109.22 165.6714 90)
+      (effects (font (size 1.27 1.27)) (justify left))
+    )
+    (property "Footprint" "Connector_Coaxial:U.FL_Molex_MCRF_73412-0110_Vertical" (id 2) (at 105.41 163.83 0)
+      (effects (font (size 1.27 1.27)) hide)
+    )
+    (property "Datasheet" "~" (id 3) (at 105.41 163.83 0)
       (effects (font (size 1.27 1.27)) hide)
     )
@@
     (pin "2")
   )
-  (symbol (lib_id "power:GND") (at 92.71 167.64 0) (unit 1)
-    (in_bom yes) (on_board yes) (fields_autoplaced)
-    (property "Reference" "#PWR0114" (id 0) (at 92.71 173.99 0)
-      (effects (font (size 1.27 1.27)) hide)
-    )
-    (property "Value" "GND" (id 1) (at 92.71 172.72 0))
-    (property "Footprint" "" (id 2) (at 92.71 167.64 0)
-      (effects (font (size 1.27 1.27)) hide)
-    )
-    (property "Datasheet" "" (id 3) (at 92.71 167.64 0)
+  (symbol (lib_id "power:GND") (at 97.79 177.8 0) (unit 1)
+    (in_bom yes) (on_board yes) (fields_autoplaced)
+    (property "Reference" "#PWR0114" (id 0) (at 97.79 184.15 0)
+      (effects (font (size 1.27 1.27)) hide)
+    )
+    (property "Value" "GND" (id 1) (at 97.79 182.88 0))
+    (property "Footprint" "" (id 2) (at 97.79 177.8 0)
+      (effects (font (size 1.27 1.27)) hide)
+    )
+    (property "Datasheet" "" (id 3) (at 97.79 177.8 0)
       (effects (font (size 1.27 1.27)) hide)
     )
@@
     )
     (pin "1")
+  )
+  (symbol (lib_id "Device:C") (at 81.28 171.45 0) (unit 1)
+    (in_bom yes) (on_board yes) (fields_autoplaced)
+    (property "Reference" "C6" (id 0) (at 85.09 170.1799 0)
+      (effects (font (size 1.27 1.27)) (justify left))
+    )
+    (property "Value" "C" (id 1) (at 85.09 172.7199 0)
+      (effects (font (size 1.27 1.27)) (justify left))
+    )
+    (property "Footprint" "Capacitor_SMD:C_0603_1608Metric_Pad1.08x0.95mm_HandSolder" (id 2) (at 82.2452 175.26 0)
+      (effects (font (size 1.27 1.27)) hide)
+    )
+    (property "Datasheet" "~" (id 3) (at 81.28 171.45 0)
+      (effects (font (size 1.27 1.27)) hide)
+    )
+    (pin "1")
+    (pin "2")
   )
   (symbol (lib_id "power:+3V3") (at 120.65 87.63 0) (unit 1)
@@
     (pin "3")
     (pin "4")
+  )
+  (symbol (lib_id "Device:R") (at 85.09 163.83 90) (unit 1)
+    (in_bom yes) (on_board yes) (fields_autoplaced)
+    (property "Reference" "R8" (id 0) (at 85.09 157.48 90))
+    (property "Value" "R" (id 1) (at 85.09 160.02 90))
+    (property "Footprint" "Resistor_SMD:R_0603_1608Metric_Pad0.98x0.95mm_HandSolder" (id 2) (at 85.09 165.608 90)
+      (effects (font (size 1.27 1.27)) hide)
+    )
+    (property "Datasheet" "~" (id 3) (at 85.09 163.83 0)
+      (effects (font (size 1.27 1.27)) hide)
+    )
+    (pin "1")
+    (pin "2")
   )
   (symbol (lib_id "RP402NX:RP402NXXXX") (at 73.66 38.1 0) (unit 1)
@@
       (reference "C5") (unit 1) (value "10u") (footprint "Capacitor_SMD:C_0805_2012Metric")
     )
+    (path "/862163c8-c6df-4776-a3a1-b3662d4f6185"
+      (reference "C6") (unit 1) (value "C") (footprint "Capacitor_SMD:C_0603_1608Metric_Pad1.08x0.95mm_HandSolder")
+    )
+    (path "/4c2ca80d-4093-4a53-8185-5c381fa3504a"
+      (reference "C7") (unit 1) (value "C") (footprint "Capacitor_SMD:C_0603_1608Metric_Pad1.08x0.95mm_HandSolder")
+    )
     (path "/fcf1cf46-cba3-4a5f-a642-24652a1181a8"
       (reference "CR1") (unit 1) (value "STTS75M2F") (footprint "STTS75M2F:STTS75M2F")
@@
       (reference "R7") (unit 1) (value "10k") (footprint "Resistor_SMD:R_0805_2012Metric")
     )
+    (path "/989d77d7-681a-4ac1-8ac8-b94744a77902"
+      (reference "R8") (unit 1) (value "R") (footprint "Resistor_SMD:R_0603_1608Metric_Pad0.98x0.95mm_HandSolder")
+    )
+    (path "/3ff58c28-e5ee-4960-9a79-47d80ed3046b"
+      (reference "R9") (unit 1) (value "R") (footprint "Resistor_SMD:R_0603_1608Metric_Pad0.98x0.95mm_HandSolder")
+    )
     (path "/43d8cc38-faad-4a4f-a2a8-32adf5b3e543"
